File: kicad_project/battery_charging.kicad_sch (KiCad schematic)
At the start: 61 parts, among them J3 USB_C_Receptacle_USB2.0, J4 Conn_01x02, U3 TVS2200DRV, U4 BQ25798RQMR, U5 TPS25750DRJKR, U6 CAT24C256

Commit message: updated gitignore
Parts:
- added JP1: Jumper_2_Open, Jumper:SolderJumper-2_P1.3mm_Open_RoundedPad1.0x1.5mm, symbol Jumper:Jumper_2_Open
- TP1: value LDO_3V3 -> FLSH_3V3
- U5: MANUFACTURER Texas Instruments -> (none); MAXIMUM_PACKAGE_HEIGHT 0.8 mm -> (none); PARTREV A -> (none); STANDARD Manufacturer Recommendations -> (none)
Connections:
- net LDO_3V3: now also JP1.2 (B); no longer C40.1, TP1.1, U6.8 (VCC)
- new net FLASH_3V3: C40.1, JP1.1 (A), TP1.1, U6.8 (VCC)
Other:
- moved on the sheet: C40
Changed lines of the file:
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@@
   (junction (at 267.97 25.4) (diameter 0) (color 0 0 0 0)
   )
+  (junction (at 101.854 166.624) (diameter 0) (color 0 0 0 0)
+  )
   (junction (at 64.77 27.94) (diameter 0) (color 0 0 0 0)
   )
@@
   (junction (at 50.8 92.71) (diameter 0) (color 0 0 0 0)
   )
+  (junction (at 77.47 161.29) (diameter 0) (color 0 0 0 0)
+  )
   (junction (at 238.76 53.34) (diameter 0) (color 0 0 0 0)
   )
@@
   )
   (junction (at 82.55 52.07) (diameter 0) (color 0 0 0 0)
-  )
-  (junction (at 104.14 161.29) (diameter 0) (color 0 0 0 0)
   )
   (junction (at 259.08 53.34) (diameter 0) (color 0 0 0 0)
@@
     (stroke (width 0) (type default))
   )
-  (wire (pts (xy 77.47 161.29) (xy 104.14 161.29))
-    (stroke (width 0) (type default))
-  )
   (wire (pts (xy 53.34 95.25) (xy 50.8 95.25))
     (stroke (width 0) (type default))
@@
     (stroke (width 0) (type default))
   )
-  (wire (pts (xy 104.14 161.29) (xy 107.95 161.29))
+  (wire (pts (xy 114.808 166.624) (xy 120.904 166.624))
     (stroke (width 0) (type default))
   )
@@
     (stroke (width 0) (type default))
   )
-  (wire (pts (xy 104.14 171.45) (xy 104.14 172.72))
+  (wire (pts (xy 101.854 177.546) (xy 101.854 178.816))
     (stroke (width 0) (type default))
   )
@@
     (stroke (width 0) (type default))
   )
+  (wire (pts (xy 79.756 160.274) (xy 77.47 160.274))
+    (stroke (width 0) (type default))
+  )
   (wire (pts (xy 254 101.6) (xy 259.08 101.6))
     (stroke (width 0) (type default))
@@
     (stroke (width 0) (type default))
   )
+  (wire (pts (xy 95.758 166.624) (xy 95.758 161.29))
+    (stroke (width 0) (type default))
+  )
   (wire (pts (xy 156.21 183.515) (xy 163.83 183.515))
     (stroke (width 0) (type default))
@@
     (stroke (width 0) (type default))
   )
+  (wire (pts (xy 101.854 166.624) (xy 101.854 169.926))
+    (stroke (width 0) (type default))
+  )
   (wire (pts (xy 41.91 135.89) (xy 53.34 135.89))
     (stroke (width 0) (type default))
@@
     (stroke (width 0) (type default))
   )
+  (wire (pts (xy 104.648 166.624) (xy 101.854 166.624))
+    (stroke (width 0) (type default))
+  )
   (wire (pts (xy 25.4 66.04) (xy 25.4 67.31))
     (stroke (width 0) (type default))
@@
     (stroke (width 0) (type default))
   )
-  (wire (pts (xy 104.14 161.29) (xy 104.14 163.83))
-    (stroke (width 0) (type default))
-  )
   (wire (pts (xy 223.52 161.29) (xy 223.52 156.21))
     (stroke (width 0) (type default))
@@
     (stroke (width 0) (type default))
   )
+  (wire (pts (xy 101.854 166.624) (xy 95.758 166.624))
+    (stroke (width 0) (type default))
+  )
   (wire (pts (xy 243.84 45.72) (xy 247.65 45.72))
     (stroke (width 0) (type default))
@@
     (stroke (width 0) (type default))
   )
+  (wire (pts (xy 95.758 161.29) (xy 77.47 161.29))
+    (stroke (width 0) (type default))
+  )
   (wire (pts (xy 55.88 185.42) (xy 63.5 185.42))
     (stroke (width 0) (type default))
@@
   )
   (wire (pts (xy 53.34 118.11) (xy 50.8 118.11))
+    (stroke (width 0) (type default))
+  )
+  (wire (pts (xy 77.47 160.274) (xy 77.47 161.29))
     (stroke (width 0) (type default))
   )
@@
     (effects (font (size 1.27 1.27)) (justify right bottom))
   )
-  (label "LDO_3V3" (at 107.95 161.29 0) (fields_autoplaced)
+  (label "LDO_3V3" (at 120.904 166.624 0) (fields_autoplaced)
     (effects (font (size 1.27 1.27)) (justify left bottom))
   )
@@
     (effects (font (size 1.27 1.27)) (justify left bottom))
   )
-  (label "LDO_3V3" (at 164.465 179.705 0) (fields_autoplaced)
+  (label "FLASH_3V3" (at 164.465 179.705 0) (fields_autoplaced)
+    (effects (font (size 1.27 1.27)) (justify left bottom))
+  )
+  (label "FLASH_3V3" (at 79.756 160.274 0) (fields_autoplaced)
     (effects (font (size 1.27 1.27)) (justify left bottom))
   )
@@
     )
   )
-  (symbol (lib_id "Device:C") (at 104.14 167.64 0) (unit 1)
+  (symbol (lib_id "Device:C") (at 101.854 173.736 0) (unit 1)
     (in_bom yes) (on_board yes) (dnp no)
-    (property "Reference" "C40" (at 107.061 166.4279 0)
-      (effects (font (size 1.27 1.27)) (justify left))
-    )
-    (property "Value" "100n" (at 107.061 168.8521 0)
-      (effects (font (size 1.27 1.27)) (justify left))
-    )
-    (property "Footprint" "Capacitor_SMD:C_0603_1608Metric" (at 105.1052 171.45 0)
-      (effects (font (size 1.27 1.27)) hide)
-    )
-    (property "Datasheet" "~" (at 104.14 167.64 0)
-      (effects (font (size 1.27 1.27)) hide)
-    )
-    (property "Digikey Part No." "1276-1000-1-ND" (at 104.14 167.64 0)
+    (property "Reference" "C40" (at 104.775 172.5239 0)
+      (effects (font (size 1.27 1.27)) (justify left))
+    )
+    (property "Value" "100n" (at 104.775 174.9481 0)
+      (effects (font (size 1.27 1.27)) (justify left))
+    )
+    (property "Footprint" "Capacitor_SMD:C_0603_1608Metric" (at 102.8192 177.546 0)
+      (effects (font (size 1.27 1.27)) hide)
+    )
+    (property "Datasheet" "~" (at 101.854 173.736 0)
+      (effects (font (size 1.27 1.27)) hide)
+    )
+    (property "Digikey Part No." "1276-1000-1-ND" (at 101.854 173.736 0)
       (effects (font (size 1.27 1.27)) hide)
     )
@@
       (effects (font (size 1.27 1.27)) (justify left))
     )
-    (property "Value" "LDO_3V3" (at 160.02 170.18 0)
+    (property "Value" "FLSH_3V3" (at 160.02 170.18 0)
       (effects (font (size 1.27 1.27)) (justify left))
     )
@@
     )
   )
-  (symbol (lib_id "power:GND") (at 104.14 172.72 0) (unit 1)
-    (in_bom yes) (on_board yes) (dnp no) (fields_autoplaced)
-    (property "Reference" "#PWR034" (at 104.14 179.07 0)
-      (effects (font (size 1.27 1.27)) hide)
-    )
-    (property "Value" "GND" (at 104.14 176.8531 0)
-      (effects (font (size 1.27 1.27)))
-    )
-    (property "Footprint" "" (at 104.14 172.72 0)
-      (effects (font (size 1.27 1.27)) hide)
-    )
-    (property "Datasheet" "" (at 104.14 172.72 0)
+  (symbol (lib_id "power:GND") (at 101.854 178.816 0) (unit 1)
+    (in_bom yes) (on_board yes) (dnp no) (fields_autoplaced)
+    (property "Reference" "#PWR034" (at 101.854 185.166 0)
+      (effects (font (size 1.27 1.27)) hide)
+    )
+    (property "Value" "GND" (at 101.854 182.9491 0)
+      (effects (font (size 1.27 1.27)))
+    )
+    (property "Footprint" "" (at 101.854 178.816 0)
+      (effects (font (size 1.27 1.27)) hide)
+    )
+    (property "Datasheet" "" (at 101.854 178.816 0)
       (effects (font (size 1.27 1.27)) hide)
     )
@@
         (path "/2045b4df-e960-493d-823c-9347bcfea953/29d2ffd5-402d-4aeb-a3f6-6081235b01c2"
           (reference "R18") (unit 1)
+        )
+      )
+    )
+  )
+  (symbol (lib_id "Jumper:Jumper_2_Open") (at 109.728 166.624 0) (unit 1)
+    (in_bom yes) (on_board yes) (dnp no) (fields_autoplaced)
+    (property "Reference" "JP1" (at 109.728 160.274 0)
+      (effects (font (size 1.27 1.27)))
+    )
+    (property "Value" "Jumper_2_Open" (at 109.728 162.814 0)
+      (effects (font (size 1.27 1.27)))
+    )
+    (property "Footprint" "Jumper:SolderJumper-2_P1.3mm_Open_RoundedPad1.0x1.5mm" (at 109.728 166.624 0)
+      (effects (font (size 1.27 1.27)) hide)
+    )
+    (property "Datasheet" "~" (at 109.728 166.624 0)
+      (effects (font (size 1.27 1.27)) hide)
+    )
+    (pin "1")
+    (pin "2")
+    (instances
+      (project "props_board_v3"
+        (path "/2045b4df-e960-493d-823c-9347bcfea953"
+          (reference "JP1") (unit 1)
+        )
+        (path "/2045b4df-e960-493d-823c-9347bcfea953/29d2ffd5-402d-4aeb-a3f6-6081235b01c2"
+          (reference "JP3") (unit 1)
         )
       )
@@
       (effects (font (size 1.27 1.27)) hide)
     )
-    (property "PARTREV" "A" (at 76.2 115.57 0)
-      (effects (font (size 1.27 1.27)) (justify bottom) hide)
-    )
-    (property "STANDARD" "Manufacturer Recommendations" (at 76.2 115.57 0)
-      (effects (font (size 1.27 1.27)) (justify bottom) hide)
-    )
-    (property "MAXIMUM_PACKAGE_HEIGHT" "0.8 mm" (at 76.2 115.57 0)
-      (effects (font (size 1.27 1.27)) (justify bottom) hide)
-    )
-    (property "MANUFACTURER" "Texas Instruments" (at 76.2 115.57 0)
-      (effects (font (size 1.27 1.27)) (justify bottom) hide)
-    )
     (property "Digikey Part No." "taobao" (at 76.2 115.57 0)
