File: kicad_project/props_board_v3.kicad_sch (KiCad schematic)
At the start: 32 parts, among them J1 Conn_01x06, J2 PWR, U1 ESP32-WROOM-32U, U2 MCP16301

Commit message: updated gitignore
Parts:
- C7: Digikey Part No. 1276-1192-1-ND1276-1192-1-ND -> 1276-1192-1-ND
Changed lines of the file:
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@@
       (effects (font (size 1.27 1.27)) hide)
     )
-    (property "Digikey Part No." "1276-1192-1-ND1276-1192-1-ND" (at 237.49 34.29 0)
+    (property "Digikey Part No." "1276-1192-1-ND" (at 237.49 34.29 0)
       (effects (font (size 1.27 1.27)) hide)
     )
